Commit message: fixed xml issue in virat.gazebo.xacro

File: models/virat/virat.gazebo.xacro (robot description, xacro)
@@ -119,16 +119,18 @@
     </gazebo>
     <gazebo reference="gps_link">
-        <plugin name="gps" filename="libhector_gazebo_ros_gps.so">
-            <alwaysOn>1</alwaysOn>
-            <updateRate>10.0</updateRate>
-            <bodyName>gps_link</bodyName>
-            <frameId>gps_link</frameId>
-            <topicName>fix</topicName>
-            <velocityTopicName>fix_velocity</velocityTopicName>
-            <drift>5.0 5.0 5.0</drift>
-            <gaussianNoise>0.1 0.1 0.1</gaussianNoise>
-            <velocityDrift>0 0 0</velocityDrift>
-            <velocityGaussianNoise>0.1 0.1 0.1</velocityGaussianNoise>
-        </plugin>
+        <sensor type="gps" name="virat_gps">
+            <plugin name="gps" filename="libhector_gazebo_ros_gps.so">
+                <alwaysOn>1</alwaysOn>
+                <updateRate>10.0</updateRate>
+                <bodyName>gps_link</bodyName>
+                <frameId>gps_link</frameId>
+                <topicName>fix</topicName>
+                <velocityTopicName>fix_velocity</velocityTopicName>
+                <drift>5.0 5.0 5.0</drift>
+                <gaussianNoise>0.1 0.1 0.1</gaussianNoise>
+                <velocityDrift>0 0 0</velocityDrift>
+                <velocityGaussianNoise>0.1 0.1 0.1</velocityGaussianNoise>
+            </plugin>
+        </sensor>
     </gazebo>
     <gazebo reference="imu_link">

File: models/virat/virat.urdf.xacro (robot description, xacro)
@@ -186,5 +186,5 @@
     <link name="imu_link">
         <visual>
-            <origin xyz="0 0 0" rpy="0 0 0"/>
+            <origin xyz="0 0 -0.13" rpy="0 0 0"/>
             <geometry>
                 <box size="0.02 0.02 0.02"/>
